Commit message: Sept 11, 2024

File: glider_hybrid_whoi_description/robots/glider_hybrid_whoi_default_kinematics.urdf.xacro (robot description, xacro)
@@ -17,5 +17,5 @@
   <xacro:arg name="inertial_reference_frame" default="world"/>
   <!-- Include the UUV macro file -->
-  <xacro:include filename="$(find glider_hybrid_whoi_description)/urdf/glider_hybrid_whoi_base_kinematics.xacro"/>
+  <xacro:include filename="$(find glider_hybrid_whoi_description)/urdf/glider_slocum_base_kinematics_slocum.xacro"/>
   <!-- Create the glider_hybrid_whoi -->
   <xacro:glider_hybrid_whoi_base
@@ -24,4 +24,4 @@
     inertial_reference_frame="$(arg inertial_reference_frame)"/>
   <!-- Joint state publisher plugin -->
-  <xacro:default_joint_state_publisher namespace="$(arg namespace)" update_rate="50"/>
+  <xacro:default_joint_state_publisher namespace="$(arg namespace)" update_rate="1"/>
 </robot>

File: glider_hybrid_whoi_description/urdf/glider_hybrid_whoi_sensors_kinematics.xacro (robot description, xacro)
@@ -62,5 +62,5 @@
       power_load="20"
       topic="${namespace}/imu/state"/>
-    <!-- Mount a camera -->
+    Mount a camera
     <xacro:regular_camera_plugin_macro
         namespace="${namespace}"

File: glider_hybrid_whoi_description/urdf/glider_slocum_base_kinematics_slocum.xacro (robot description, xacro)
@@ -18,13 +18,14 @@
   <xacro:include filename="$(find uuv_gazebo_ros_plugins)/urdf/snippets.xacro"/>
   <!-- Properties -->
-  <xacro:property name="mass" value="56.0"/>
+  <xacro:property name="mass" value="69.25"/>
   <xacro:property name="fluid_density" value="1024.0"/>
   <xacro:property name="gravity" value="9.81"/>
   <xacro:property name="cob" value="0 0 0"/>
   <xacro:property name="cog" value="0 0 0.0054"/>
-  <xacro:property name="visual_mesh_file" value="file://$(find glider_hybrid_whoi_description)/mesh/glider_hybrid_whoi/glider_hybrid_whoi_body.dae" />
-  <xacro:property name="collision_mesh_file" value="file://$(find glider_hybrid_whoi_description)/mesh/glider_hybrid_whoi/glider_hybrid_whoi_collision.dae" />
-  <xacro:property name="left_prop_mesh_file" value="file://$(find glider_hybrid_whoi_description)/mesh/glider_hybrid_whoi/glider_hybrid_whoi_left_propeller.dae" />
-  <xacro:property name="right_prop_mesh_file" value="file://$(find glider_hybrid_whoi_description)/mesh/glider_hybrid_whoi/glider_hybrid_whoi_right_propeller.dae" />
+  <xacro:property name="visual_mesh_file" value="file://$(find glider_hybrid_whoi_description)/mesh/glider_slocum/Slocum-Glider.dae" />
+  <xacro:property name="collision_mesh_file" value="file://$(find glider_hybrid_whoi_description)/mesh/glider_slocum/COLLISION-Slocum-Glider.dae" />
+  <xacro:property name="prop_mesh_file" value="file://$(find glider_hybrid_whoi_description)/mesh/glider_slocum/Slocum-Glider-Propeller.dae" />
+  <!-- <xacro:property name="left_fin_mesh_file" value="file://$(find glider_hybrid_whoi_description)/mesh/glider_slocum/Slocum-Glider-LeftFin.dae" /> -->
+  <!-- <xacro:property name="right_fin_mesh_file" value="file://$(find glider_hybrid_whoi_description)/mesh/glider_slocum/Slocum-Glider-RightFin.dae" /> -->
   <xacro:macro name="glider_hybrid_whoi_base" params="namespace debug inertial_reference_frame">
     <!-- Base_link of the model -->
@@ -45,5 +46,5 @@
         <mass value="${mass}"/>
         <origin xyz="0 0 0" rpy="0 0 0" />
-        <inertia ixx="0.3048" ixy="0" ixz="0" iyy="13.976" iyz="0" izz="13.976" />
+        <inertia ixx="10" ixy="0" ixz="0" iyy="10" iyz="0" izz="10" />
       </inertial>
     </link>
@@ -53,9 +54,9 @@
       <dynamics>
         <type>FirstOrder</type>
-        <timeConstant>0.0</timeConstant>
+        <timeConstant>0.1</timeConstant>
       </dynamics>
       <conversion>
         <type>Basic</type>
-        <rotorConstant>0.0</rotorConstant>
+        <rotorConstant>4.9e-05</rotorConstant>
       </conversion>
     </xacro:property>
@@ -74,5 +75,5 @@
     <xacro:property name="thruster_id" value="1"/>
     <joint name="${namespace}/thruster_${thruster_id}_joint" type="continuous">
-      <origin xyz="-0.558 -0.05 0" rpy="0 0 -${0.07*pi}"/>
+      <origin xyz="0.0 0.0 0" rpy="0 0 0"/>
       <axis xyz="1 0 0"/>
       <parent link="${namespace}/base_link"/>
@@ -82,7 +83,7 @@
       <xacro:insert_block name="dummy_link_properties_for_visual_rotation"/>
       <visual>
-        <origin xyz="0.541 0.12 0" rpy="0 0 -${0.46*pi}"/>
-        <geometry>
-          <mesh filename="${right_prop_mesh_file}" scale="1 1 1"/>
+        <origin xyz="0 0 0" rpy="0 0 -${0.46*pi}"/>
+        <geometry>
+          <mesh filename="${prop_mesh_file}" scale="1 1 1"/>
         </geometry>
       </visual>
@@ -99,32 +100,96 @@
       <selfCollide>false</selfCollide>
     </gazebo>
-    <!-- Second propeller -->
-    <xacro:property name="thruster_id" value="0"/>
-    <joint name="${namespace}/thruster_${thruster_id}_joint" type="continuous">
-      <origin xyz="-0.558 0.05 0" rpy="0 0 ${0}"/>
-      <axis xyz="1 0 0"/>
-      <parent link="${namespace}/base_link"/>
-      <child link="${namespace}/thruster_${thruster_id}"/>
-    </joint>
-    <link name="${namespace}/thruster_${thruster_id}">
-      <xacro:insert_block name="dummy_link_properties_for_visual_rotation"/>
-      <visual>
-        <origin xyz="-0.541 0.12 0" rpy="0 0 ${0.46*pi}"/>
-        <geometry>
-          <mesh filename="${left_prop_mesh_file}" scale="1 1 1"/>
-        </geometry>
-      </visual>
-    </link>
-    <gazebo>
-      <plugin name="${namespace}_${thruster_id}_thruster_model" filename="libuuv_thruster_ros_plugin.so">
-        <linkName>${namespace}/thruster_${thruster_id}</linkName>
-        <jointName>${namespace}/thruster_${thruster_id}_joint</jointName>
-        <thrusterID>${thruster_id}</thrusterID>
-        <xacro:insert_block name="dummy_plugin_properties_for_visual_rotation"/>
-      </plugin>
-    </gazebo>
-    <gazebo reference="${namespace}/thruster_${thruster_id}">
+    <!-- add a small cube to repersent a hydrophone on the gliders wing -->
+    <xacro:property name="hydrophone_4_id" value="4"/>
+    <link name="${namespace}/hydrophone_${hydrophone_4_id}">
+      <visual>
+        <geometry>
+          <box size="0.2 0.05 0.05"/>
+        </geometry>
+      </visual>
+      <collision>
+        <geometry>
+          <box size="0.2 0.05 0.05"/>
+        </geometry>
+      </collision>
+      <inertial>
+        <mass value="0.5"/>
+        <inertia ixx="0.1" ixy="0" ixz="0" iyy="0.1" iyz="0" izz="0.1"/>
+      </inertial>
+    </link>
+    <joint name="${namespace}/hydrophone_${hydrophone_4_id}_joint" type="continuous">
+      <origin xyz="-0.3 1.1 0.03" rpy="0 0 0"/>
+      <parent link="${namespace}/base_link"/>
+      <child link="${namespace}/hydrophone_${hydrophone_4_id}"/>
+    </joint>
+    <gazebo reference="$hydrophone_${hydrophone_4_id}">
       <selfCollide>false</selfCollide>
     </gazebo>
+    <!-- add a small cube to repersent a hydrophone on the gliders wing -->
+    <link name="${namespace}/hydrophone_3">
+      <visual>
+        <geometry>
+          <box size="0.2 0.05 0.05"/>
+        </geometry>
+      </visual>
+      <collision>
+        <geometry>
+          <box size="0.2 0.05 0.05"/>
+        </geometry>
+      </collision>
+      <inertial>
+        <mass value="0.5"/>
+        <inertia ixx="0.1" ixy="0" ixz="0" iyy="0.1" iyz="0" izz="0.1"/>
+      </inertial>
+    </link>
+    <joint name="${namespace}/hydrophone_3_joint" type="continuous">
+      <origin xyz="-0.3 -1.1 0.03" rpy="0 0 0"/>
+      <parent link="${namespace}/base_link"/>
+      <child link="${namespace}/hydrophone_3"/>
+    </joint>
+      <!-- add a small cube to repersent a hydrophone on the gliders wing -->
+    <link name="${namespace}/hydrophone_1">
+      <visual>
+        <geometry>
+          <box size="0.3 0.1 0.1"/>
+        </geometry>
+      </visual>
+      <collision>
+        <geometry>
+          <box size="0.3 0.1 0.1"/>
+        </geometry>
+      </collision>
+      <inertial>
+        <mass value="0.8"/>
+        <inertia ixx="0.1" ixy="0" ixz="0" iyy="0.1" iyz="0" izz="0.1"/>
+      </inertial>
+    </link>
+    <joint name="${namespace}/hydrophone_1_joint" type="continuous">
+      <origin xyz="1.0 0.0 0.25" rpy="0 0 0"/>
+      <parent link="${namespace}/base_link"/>
+      <child link="${namespace}/hydrophone_1"/>
+    </joint>
+        <!-- add a small cube to repersent a hydrophone on the gliders wing -->
+    <link name="${namespace}/hydrophone_2">
+      <visual>
+        <geometry>
+          <box size="0.2 0.05 0.05"/>
+        </geometry>
+      </visual>
+      <collision>
+        <geometry>
+          <box size="0.2 0.05 0.05"/>
+        </geometry>
+      </collision>
+      <inertial>
+        <mass value="0.5"/>
+        <inertia ixx="0.1" ixy="0" ixz="0" iyy="0.1" iyz="0" izz="0.1"/>
+      </inertial>
+    </link>
+    <joint name="${namespace}/hydrophone_2_joint" type="continuous">
+      <origin xyz="-1.0 0.0 0.25" rpy="0 0 0"/>
+      <parent link="${namespace}/base_link"/>
+      <child link="${namespace}/hydrophone_2"/>
+    </joint>
     <!-- Kinematics Plugin -->
     <gazebo>
@@ -154,14 +219,14 @@
           <topic_stratified_database>stratified_current_velocity_database</topic_stratified_database>
           <velocity_north>
-            <noiseAmp>0.3</noiseAmp>
-            <noiseFreq>0.0</noiseFreq>
+            <noiseAmp>0.7</noiseAmp>
+            <noiseFreq>0.1</noiseFreq>
           </velocity_north>
           <velocity_east>
-            <noiseAmp>0.3</noiseAmp>
-            <noiseFreq>0.0</noiseFreq>
+            <noiseAmp>0.7</noiseAmp>
+            <noiseFreq>0.1</noiseFreq>
           </velocity_east>
           <velocity_down>
-            <noiseAmp>0.3</noiseAmp>
-            <noiseFreq>0.0</noiseFreq>
+            <noiseAmp>0.7</noiseAmp>
+            <noiseFreq>0.1</noiseFreq>
           </velocity_down>
         </transient_current>
