Commit message: push

File: glider_hybrid_whoi_description/urdf/glider_slocum_base_kinematics_slocum.xacro (robot description, xacro)
@@ -85,5 +85,5 @@
         <origin xyz="0 0 0" rpy="0 0 -${0.46*pi}"/>
         <geometry>
-          <mesh filename="${prop_mesh_file}" scale="1 1 1"/>
+          <mesh filename="${prop_mesh_file}" scale="0 0 0"/>
         </geometry>
       </visual>
@@ -119,5 +119,5 @@
     </link>
     <joint name="${namespace}/hydrophone_${hydrophone_4_id}_joint" type="continuous">
-      <origin xyz="-0.3 1.1 0.03" rpy="0 0 0"/>
+      <origin xyz="-0.6 0.47219 0.03" rpy="0 0 0"/>
       <parent link="${namespace}/base_link"/>
       <child link="${namespace}/hydrophone_${hydrophone_4_id}"/>
@@ -144,5 +144,5 @@
     </link>
     <joint name="${namespace}/hydrophone_3_joint" type="continuous">
-      <origin xyz="-0.3 -1.1 0.03" rpy="0 0 0"/>
+      <origin xyz="-0.6 -0.47219 0.03" rpy="0 0 0"/>
       <parent link="${namespace}/base_link"/>
       <child link="${namespace}/hydrophone_3"/>
@@ -152,5 +152,5 @@
       <visual>
         <geometry>
-          <box size="0.3 0.1 0.1"/>
+          <box size="0.5 0.1 0.1"/>
         </geometry>
       </visual>
@@ -170,5 +170,5 @@
       <child link="${namespace}/hydrophone_1"/>
     </joint>
-        <!-- add a small cube to repersent a hydrophone on the gliders wing -->
+        <!-- Hydrophone on tail -->
     <link name="${namespace}/hydrophone_2">
       <visual>
@@ -188,5 +188,5 @@
     </link>
     <joint name="${namespace}/hydrophone_2_joint" type="continuous">
-      <origin xyz="-1.0 0.0 0.25" rpy="0 0 0"/>
+      <origin xyz="-1.32791 -0.04064 0.25" rpy="0 0 0"/>
       <parent link="${namespace}/base_link"/>
       <child link="${namespace}/hydrophone_2"/>

Commit message: Test -MM

File: glider_hybrid_whoi_description/urdf/glider_slocum_base_kinematics_slocum.xacro (robot description, xacro)
@@ -192,4 +192,28 @@
       <child link="${namespace}/hydrophone_2"/>
     </joint>
+      <!-- Add a rudder on the taial that will move -->
+    <!-- <link name="${namespace}/rudder">
+      <collision>
+        <geometry>
+          <box size="0.3 0.1 0.1"/>
+        </geometry>
+      </collision>
+      <inertial>
+        <mass value="0.8"/>
+        <inertia ixx="0.1" ixy="0" ixz="0" iyy="0.1" iyz="0" izz="0.1"/>
+      </inertial>
+      <visual>
+        <geometry>
+          <box size="0.3 0.1 0.1"/>
+        </geometry>
+      </visual>
+    </link>
+    <joint name="${namespace}/yaw_fin_joint" type="revolute">
+      <parent link="${namespace}/base_link"/>
+      <child link="${namespace}/rudder"/>
+      <origin xyz="0 0 0.05" rpy="0 0 0"/>
+      <axis xyz="0 0 1"/>
+      <limit lower="-1.57" upper="1.57" effort="10" velocity="1.0"/>
+    </joint> -->
     <!-- Kinematics Plugin -->
     <gazebo>
@@ -234,13 +258,13 @@
       </plugin>
     </gazebo>
-    <gazebo>
+    <!-- <gazebo>
       <plugin name="gazebo_ros_control" filename="libgazebo_ros_control.so">
         <robotNamespace>/${namespace}</robotNamespace>
-        <robotParam>/${namespace}/robot_description</robotParam>
+        <robotParam>${namespace}/robot_description</robotParam>
         <bathymetry>
           <interval_s>1.0</interval_s>
         </bathymetry>
       </plugin>
-    </gazebo>
+    </gazebo> -->
     <!-- TODO: Parametrize the battery unit -->
     <xacro:basic_linear_battery_macro

File: glider_hybrid_whoi_description/urdf/uw_hector_imu_plugin.xacro (robot description, xacro)
@@ -40,5 +40,5 @@
                 <robotNamespace>${namespace}</robotNamespace>
                 <serviceName>hector_imu/is_calibrated</serviceName>
-                <gaussianNoise>0.001</gaussianNoise>
+                <gaussianNoise>0.1</gaussianNoise>
                 <xyzOffset>0</xyzOffset>
                 <xyzOffset>0</xyzOffset>
